File: E10.kicad_pcb (KiCad board)
At the start: 2 copper layers, 79.4 x 21.6 mm, 45 parts, among them J1 LED 8-15, J2 WS-bus output, J3 WS-bus input, J4 UPDI, J5 Debug, J6 LED common, J7 LED 0-7, J8 LED Common, U1 AVR-64da32, U2 MIC5205-5.0YM5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

Commit message: mod: optimized for PCB assembly
Parts:
- D1, R20, R23: moved to F.Cu
- moved D1 62.3 mm to (102.4, 94.4), turned to 90 degrees
- moved R20 3.62 mm to (127.0, 95.8), turned to 180 degrees
- moved R23 2.87 mm to (153.0, 85.5), turned to 270 degrees
- moved R24 0.93 mm to (155.9, 85.5)
- moved U3 0.93 mm to (158.5, 85.6)
- moved R25 0.93 mm to (154.4, 85.5)
Routing:
- net +5V: track 135.6 -> 154.1 mm
- net VDD: track 17.3 -> 12.9 mm, vias 3 -> 2
- net Net-(JP2-Pad1): track 8.66 -> 12.9 mm, vias 2 -> 1
- net DAC: track 34.6 -> 36.8 mm, vias 2 -> 3
- net Net-(D2-Pad2): track 0.00 -> 2.05 mm
- net GND: vias 10 -> 11
Other:
- board text added: "E10.3"
- board text removed: "E10.2"
